Commit message: Fix URDF/SRDF to work with MoveIt!

File: ur_description/urdf/ur5_joint_limited_robot.urdf.xacro (robot description, xacro)
@@ -15,7 +15,7 @@
     wrist_3_lower_limit="${-pi}" wrist_3_upper_limit="${pi}"
   />
-  <link name="world" />
-  <joint name="world_joint" type="fixed">
-    <parent link="world" />
+  <link name="base_link_no_inertia" />
+  <joint name="base_link_no_inertia_joint" type="fixed">
+    <parent link="base_link_no_inertia" />
     <child link = "base_link" />
     <origin xyz="0.0 0.0 0.0" rpy="0.0 0.0 0.0" />

File: ur_description/urdf/ur5_robot.urdf.xacro (robot description, xacro)
@@ -8,7 +8,7 @@
   <!-- arm -->
   <xacro:ur5_robot prefix="" joint_limited="false"/>
-  <link name="world" />
-  <joint name="world_joint" type="fixed">
-    <parent link="world" />
+  <link name="base_link_no_inertia" />
+  <joint name="base_link_no_inertia_joint" type="fixed">
+    <parent link="base_link_no_inertia" />
     <child link = "base_link" />
     <origin xyz="0.0 0.0 0.0" rpy="0.0 0.0 0.0" />
